File: myteensy32.kicad_pcb (KiCad board)
At the start: 2 copper layers, 35.6 x 17.8 mm, 31 parts, among them J1 Conn_01x14_Male, J2 Conn_01x14_Male, J3 USB_C_Receptacle_USB2.0, SW1 RESET, SW2 PROG, U1 MKL04Z32VLC4, U2 MK20DX256VLH7, U3 MCP2562-E-SN, U4 NJM2884U1, Y2 16MHz

Commit message: すべてを削除してネットリストの再読み込み
Parts:
- C1, C10, C2, C3, C4, C9, D1, D2, J1, J2, R1, R2, R3, R4, R5, U3, U4: moved to F.Cu
- moved J1 55.7 mm to (95.5, 61.3), turned to 0 degrees
- moved SW2 43.1 mm to (107.5, 75.1), turned to 0 degrees
- moved R5 42.7 mm to (108.7, 87.9)
- moved SW1 41.9 mm to (107.5, 79.4), turned to 0 degrees
- moved C5 41.1 mm to (100.1, 88.1), turned to 0 degrees
- moved R3 39.5 mm to (104.3, 90.8), turned to 0 degrees
- moved U2 39.3 mm to (104.8, 65.9), turned to 0 degrees
- moved C3 38.2 mm to (103.9, 93.8)
- moved J2 37.9 mm to (90.9, 61.3), turned to 0 degrees
- moved D4 37.1 mm to (112.6, 77.9)
- moved R2 35.2 mm to (108.8, 85.3), turned to 0 degrees
- moved Y2 34.4 mm to (100.1, 80.5)
- moved D1 27.8 mm to (100.1, 84.3), turned to 0 degrees
- moved D2 26.9 mm to (104.5, 84.3), turned to 0 degrees
- moved R4 26.4 mm to (99.9, 93.8)
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Routing:
- net GND: track 109.8 -> 0.00 mm, vias 9 -> 0
- net +3V3: track 87.3 -> 0.00 mm, vias 5 -> 0
- net /RESET: track 36.2 -> 0.00 mm, vias 3 -> 0
- net /USB-: track 36.1 -> 0.00 mm
- net /ProgramModeBtn: track 35.5 -> 0.00 mm, vias 2 -> 0
- net /USB+: track 33.3 -> 0.00 mm
- net Net-(J2-Pad9): track 31.1 -> 0.00 mm, vias 1 -> 0
- net Net-(J2-Pad4): track 30.0 -> 0.00 mm, vias 1 -> 0
- net Net-(J2-Pad7): track 29.4 -> 0.00 mm, vias 1 -> 0
- net +5V: track 28.6 -> 0.00 mm, vias 2 -> 0
- net Net-(J2-Pad8): track 28.2 -> 0.00 mm, vias 1 -> 0
- net Net-(J2-Pad2): track 27.8 -> 0.00 mm, vias 1 -> 0
- net Net-(J1-Pad11): track 26.9 -> 0.00 mm, vias 1 -> 0
- net Net-(J2-Pad3): track 26.2 -> 0.00 mm, vias 1 -> 0
- net Net-(J1-Pad10): track 25.8 -> 0.00 mm, vias 1 -> 0
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- removed copper zone on B.Cu, net GND
- removed copper zone on F.Cu, net GND
Other:
- board outline removed

Commit message: wideな感じで配線してみる
Parts:
- added H1: MountingHole, mylib:Hole_3.2mm_NPTH, F.Cu at (112.2, 54.0)
- added H2: MountingHole, mylib:Hole_3.2mm_NPTH, F.Cu at (162.2, 54.0)
- added H3: MountingHole, mylib:Hole_3.2mm_NPTH, F.Cu at (112.2, 104.0)
- added H4: MountingHole, mylib:Hole_3.2mm_NPTH, F.Cu at (162.2, 104.0)
- added J4: Conn_01x14_Male, Connector_PinHeader_2.54mm:PinHeader_1x14_P2.54mm_Vertical, F.Cu at (226.1, 62.5)
- added J5: Conn_01x14_Male, Connector_PinHeader_2.54mm:PinHeader_1x14_P2.54mm_Vertical, F.Cu at (203.3, 95.5)
- added J6: Conn_01x14_Male, Connector_PinHeader_2.54mm:PinHeader_1x14_P2.54mm_Vertical, F.Cu at (233.7, 47.3)
- added J7: Conn_01x07_Male, Connector_PinSocket_2.54mm:PinSocket_1x07_P2.54mm_Vertical, F.Cu at (222.3, 52.4)
- moved J1 128.1 mm to (223.6, 62.5)
- moved J2 119.9 mm to (205.8, 95.5), turned to 180 degrees
- moved Y2 115.2 mm to (214.7, 68.9), turned to 180 degrees
- moved C6 113.3 mm to (217.7, 86.4), turned to 180 degrees
- moved U2 110.5 mm to (214.7, 77.8), turned to 135 degrees
- moved J3 101.2 mm to (211.7, 89.0)
- moved F1 93.1 mm to (213.3, 86.4), turned to 180 degrees
- moved U1 85.7 mm to (214.7, 61.2), turned to 315 degrees
- moved C1 85.6 mm to (37.2, 81.6)
- moved C11 85.6 mm to (31.6, 87.9)
- moved C2 85.6 mm to (31.9, 90.4)
- moved C4 85.6 mm to (41.2, 81.6)
- moved C7 85.6 mm to (51.8, 70.2)
- moved C8 85.6 mm to (37.2, 84.2)
- moved C10 74.3 mm to (30.1, 66.0)
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Routing:
- net GND: track 0.00 -> 19.7 mm
- net Net-(C6-Pad2): track 0.00 -> 13.4 mm
- net Net-(R3-Pad2): track 0.00 -> 4.64 mm
- net Net-(R2-Pad2): track 0.00 -> 3.48 mm
- net Net-(J2-Pad9): track 0.00 -> 2.54 mm
- net Net-(J2-Pad8): track 0.00 -> 2.54 mm
- net Net-(J2-Pad7): track 0.00 -> 2.54 mm
- net Net-(J2-Pad4): track 0.00 -> 2.54 mm
- net Net-(J2-Pad3): track 0.00 -> 2.54 mm
- net Net-(J2-Pad2): track 0.00 -> 2.54 mm
- net Net-(J2-Pad14): track 0.00 -> 2.54 mm
- net Net-(J2-Pad13): track 0.00 -> 2.54 mm
- net Net-(J2-Pad12): track 0.00 -> 2.54 mm
- net Net-(J2-Pad11): track 0.00 -> 2.54 mm
- net Net-(J2-Pad10): track 0.00 -> 2.54 mm
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Other:
- board outline added: 120.2 x 60 mm
